Commit message: Current urdf model
git-svn-id: https://roboticssrv.wtb.tue.nl/svn/ros/user/Janno/tue_calibration@24064 3a3c2cfb-d3b9-409e-9e75-db8fcdbcaac6

File: urdf/amigo.urdf (robot description, URDF)
Before this commit: robot amigo, 76 links, 75 joints
Links:
- added link opt_head_mount_vertical, mass 0.001
- added link opt_neck_lateral, mass 0.001
- added link opt_neck_length, mass 0.001
- added link opt_neck_rot, mass 0.001
- added link opt_tilt, mass 0.001
Joints:
- added joint opt_head_mount_vertical_joint: type prismatic, parent opt_head_mount, child opt_head_mount_vertical, origin xyz=0.0 0.0 0.0 rpy=0.0 0.0 0.0, axis 1 0 0, limit lower=-0.25 upper=0.25 effort=1000 velocity=1.0
- added joint opt_neck_lateral_joint: type prismatic, parent opt_neck_length, child opt_neck_lateral, origin xyz=0.0 0.0 0.0 rpy=0.0 0.0 0.0, axis 0 1 0, limit lower=-0.25 upper=0.25 effort=1000 velocity=1.0
- added joint opt_neck_length_joint: type fixed, parent opt_tilt, child opt_neck_length, origin xyz=0.0 0.0 0.0 rpy=0.0 0.0 0.0, axis 0 0 1, limit lower=-0.25 upper=0.25 effort=1000 velocity=1.0
- added joint opt_neck_rot_joint: type revolute, parent opt_neck_lateral, child opt_neck_rot, origin xyz=0.0 0.0 0.0 rpy=0.0 0.0 0.0, axis 0 0 1, limit lower=-0.25 upper=0.25 effort=1000 velocity=1.0
- added joint opt_tilt_joint: type revolute, parent head, child opt_tilt, origin xyz=0.0 0.0 0.0 rpy=0.0 0.0 0.0, axis 0 1 0, limit lower=-0.25 upper=0.25 effort=1000 velocity=1.0
- joint head_mount_joint: child opt_head_mount -> head_mount; origin xyz=0.0 0.0 0.0 rpy=  0.0 0.0 0.0 -> xyz=0.11 0.0 0.0426 rpy=-0.07 0.0 0.0; parent torso -> opt_head_mount_vertical
- joint opt_head_mount_joint: axis 1 0 0 -> 0 0 1; child head_mount -> opt_head_mount; parent opt_head_mount -> torso
- joint top_kinect/base_kinect_joint: origin xyz=0.07 0.05 0.10 rpy=0.02 0.05 0.015 -> xyz=0.035 0.0 0.10 rpy=0.0 0.0 0.05; parent head -> opt_neck_rot

Commit message: First update
git-svn-id: https://roboticssrv.wtb.tue.nl/svn/ros/user/Janno/tue_calibration@24075 3a3c2cfb-d3b9-409e-9e75-db8fcdbcaac6

File: urdf/amigo.urdf (robot description, URDF)
Before this commit: robot amigo, 81 links, 80 joints
Joints:
- joint head_mount_joint: origin xyz=0.11 0.0 0.0426 rpy=-0.07 0.0 0.0 -> xyz=0.085 0.0 0.0846 rpy=-0.07 0.0 0.0
- joint neck_tilt_joint: origin xyz=0.0 0.0 0.0445 rpy=0.0 0.0 0.0 -> xyz=0.0 0.0 0.0445 rpy=0.0 0.02 0.0
- joint top_kinect/base_kinect_joint: origin xyz=0.035 0.0 0.10 rpy=0.0 0.0 0.05 -> xyz=0.035 0.0078 0.10 rpy=0.0 0.0 0.077
