Commit message: Elaborated testnode, algorithm seems to work
git-svn-id: https://roboticssrv.wtb.tue.nl/svn/ros/user/Janno/tue_calibration@24168 3a3c2cfb-d3b9-409e-9e75-db8fcdbcaac6

File: test/amigo24127mod.urdf (robot description, URDF)
Before this commit: robot amigo, 75 links, 74 joints
Joints:
- joint head_mount_joint: origin xyz=0.097 0.0 0.0 rpy=  0.0 0.0 0.0 -> xyz=0.097 0.0 0.426 rpy=0.0 0.0 0.0
- joint top_kinect/base_kinect_joint: origin xyz=0.07 0.05 0.10 rpy=0.02 0.05 0.015 -> xyz=0.07 0.035 0.10 rpy=0.02 0.05 0.015

File: test/amigo24127opt.urdf (robot description, URDF)
Before this commit: robot amigo, 75 links, 74 joints
Links:
- added link opt_head_mount, mass 0.001
- added link opt_neck_lateral, mass 0.001
Joints:
- added joint opt_head_mount_joint: type prismatic, parent torso, child opt_head_mount, origin xyz=0.0 0.0 0.0 rpy=0.0 0.0 0.0, axis 0 0 1, limit lower=-0.25 upper=0.25 effort=1000 velocity=1.0
- added joint opt_neck_lateral_joint: type prismatic, parent head, child opt_neck_lateral, origin xyz=0.0 0.0 0.0 rpy=0.0 0.0 0.0, axis 0 1 0, limit lower=-0.25 upper=0.25 effort=1000 velocity=1.0
- joint head_mount_joint: parent torso -> opt_head_mount
- joint top_kinect/base_kinect_joint: parent head -> opt_neck_lateral

Commit message: Added some test results
git-svn-id: https://roboticssrv.wtb.tue.nl/svn/ros/user/Janno/tue_calibration@24317 3a3c2cfb-d3b9-409e-9e75-db8fcdbcaac6

File: test/amigo24127mod.urdf (robot description, URDF)
Before this commit: robot amigo, 75 links, 74 joints
Joints:
- joint head_mount_joint: origin xyz=0.097 0.0 0.426 rpy=0.0 0.0 0.0 -> xyz=0.097 0.0 0.0426 rpy=0.0 0.0 0.0
- joint neck_tilt_joint: origin xyz=0.0 0.0 0.0445 rpy=0.0 0.0 0.0 -> xyz=0.0 0.0 0.0445 rpy=0.0 0.0 0.01
- joint top_kinect/base_kinect_joint: origin xyz=0.07 0.035 0.10 rpy=0.02 0.05 0.015 -> xyz=0.07 0.05 0.10 rpy=0.02 0.05 0.015

File: test/amigo24127opt.urdf (robot description, URDF)
Before this commit: robot amigo, 77 links, 76 joints
Links:
- added link opt_head_mount_vertical, mass 0.001
- added link opt_tilt, mass 0.001
Joints:
- added joint opt_head_mount_vertical_joint: type prismatic, parent opt_head_mount, child opt_head_mount_vertical, origin xyz=0.0 0.0 0.0 rpy=0.0 0.0 0.0, axis 1 0 0, limit lower=-0.25 upper=0.25 effort=1000 velocity=1.0
- added joint opt_tilt_joint: type revolute, parent head, child opt_tilt, origin xyz=0.0 0.0 0.0 rpy=0.0 0.0 0.0, axis 0 1 0, limit lower=-0.25 upper=0.25 effort=1000 velocity=1.0
- joint head_mount_joint: parent opt_head_mount -> opt_head_mount_vertical
- joint opt_neck_lateral_joint: parent head -> opt_tilt; type prismatic -> fixed
